File: 71kHzTransmitter.kicad_sch (KiCad schematic)
At the start: 26 parts, among them Q1 ZTX603, U1 4046, U2 LM324

Commit message: fixed models for more accurate/useable sim
Parts:
- added MES?: Oscilloscope, symbol Device:Oscilloscope
- C5: footprint Package_SO:SOIC-8_3.9x4.9mm_P1.27mm -> (none)
- R1: value 39.46k -> 49.7k
Connections:
- net 4.5V renamed VREF

Commit message: TSAL6100 Name Change
Parts:
- removed MES?: Oscilloscope, symbol Device:Oscilloscope
- D1: value TSAL4400 -> TSAL6100
Changed lines of the file:
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@@
-	)
-	(symbol
-		(lib_id "Device:Oscilloscope")
-		(at 115.57 66.675 0)
-		(unit 1)
-		(body_style 1)
-		(exclude_from_sim no)
-		(in_bom yes)
-		(on_board yes)
-		(in_pos_files yes)
-		(dnp no)
-		(fields_autoplaced yes)
-		(property "Reference" "MES?"
-			(at 119.38 64.7064 0)
-			(show_name no)
-			(do_not_autoplace no)
-			(effects
-				(font
-					(size 1.27 1.27)
-				)
-				(justify left)
-			)
-		)
-		(property "Value" "Oscilloscope"
-			(at 119.38 67.2464 0)
-			(show_name no)
-			(do_not_autoplace no)
-			(effects
-				(font
-					(size 1.27 1.27)
-				)
-				(justify left)
-			)
-		)
-		(property "Footprint" ""
-			(at 115.57 64.135 90)
-			(hide yes)
-			(show_name no)
-			(do_not_autoplace no)
-			(effects
-				(font
-					(size 1.27 1.27)
-				)
-			)
-		)
-		(property "Datasheet" ""
-			(at 115.57 64.135 90)
-			(hide yes)
-			(show_name no)
-			(do_not_autoplace no)
-			(effects
-				(font
-					(size 1.27 1.27)
-				)
-			)
-		)
-		(property "Description" "Oscilloscope"
-			(at 115.57 66.675 0)
-			(hide yes)
-			(show_name no)
-			(do_not_autoplace no)
-			(effects
-				(font
-					(size 1.27 1.27)
-				)
-			)
-		)
-		(pin "1"
-		)
-		(pin "2"
-		)
-		(instances
-			(project "71kHzTransmitter"
-				(path "/9d28fa65-b7fa-4b75-a49b-191561a10239"
-					(reference "MES?")
-					(unit 1)
-				)
-			)
-		)
 	)
 	(symbol
@@
 			)
 		)
-		(property "Value" "TSAL4400"
+		(property "Value" "TSAL6100"
 			(at 152.4 157.9879 90)
 			(show_name no)

Commit message: Decoupling Caps
Parts:
- added C8, C9: 100n, Capacitor_THT:C_Disc_D5.0mm_W2.5mm_P5.00mm, symbol Device:C_Small
- C1: footprint Package_SO:SOIC-8_3.9x4.9mm_P1.27mm -> Capacitor_THT:C_Rect_L7.0mm_W2.5mm_P5.00mm
- C2, C6, C7: footprint (none) -> Capacitor_THT:C_Disc_D5.0mm_W2.5mm_P5.00mm
- C3: footprint Package_SO:SOIC-8_3.9x4.9mm_P1.27mm -> Capacitor_THT:CP_Radial_D10.0mm_P5.00mm
- C4: footprint Package_SO:SOIC-8_3.9x4.9mm_P1.27mm -> Capacitor_THT:C_Disc_D5.0mm_W2.5mm_P5.00mm
- C5: footprint (none) -> Capacitor_THT:CP_Radial_D6.3mm_P2.50mm
- D1: footprint LED_THT:LED_D3.0mm_IRBlack -> LED_THT:LED_D5.0mm_IRBlack
- R1, R4, R6, R7, R8, R9: footprint (none) -> Resistor_THT:R_Axial_DIN0207_L6.3mm_D2.5mm_P7.62mm_Horizontal
- R10, R11, R12, R2: footprint Package_DIP:DIP-8_W7.62mm -> Resistor_THT:R_Axial_DIN0207_L6.3mm_D2.5mm_P7.62mm_Horizontal
- R3: footprint Package_DIP:DIP-8_W7.62mm -> Resistor_THT:R_Axial_DIN0309_L9.0mm_D3.2mm_P10.16mm_Horizontal
- RV1, RV2: footprint (none) -> Potentiometer_THT:Potentiometer_Runtron_RM-065_Vertical
- U1: footprint (none) -> Package_DIP:DIP-16_W7.62mm
- U2: footprint Package_DFN_QFN:QFN-16-1EP_3x3mm_P0.5mm_EP1.7x1.7mm -> Package_DIP:DIP-14_W7.62mm
- V1, V2: now left out of the parts list
Connections:
- net +9V: now also C8.1, C9.1
- net GND: now also C8.2, C9.2
Other:
- note added: "Decoupling Cap (place near U1)"
- note added: "Decoupling Cap (place near U2)"
- moved on the sheet: U2E
